Commit message: Version : V 0.1.0.0
Update :
1. REFINE code.

File: legged-gym/resources/robots/gr1t1/urdf/GR1T1_lower_limb.urdf (robot description, URDF)
Before this commit: robot GR1T1, 33 links, 32 joints
Links:
- added link z_link_imu; visual box size=0.05 0.05 0.02
Joints:
- added joint z_joint_imu: type fixed, parent base, child z_link_imu, origin xyz=-0.0648 0 -0.1015 rpy=0 0 0
- joint head_pitch: type revolute -> fixed
- joint head_roll: type revolute -> fixed
- joint head_yaw: type revolute -> fixed
- joint l_ankle_pitch: limit lower=-1.05 upper=0.52 effort=8 velocity=20.32 -> lower=-1.05 upper=0.52 effort=16 velocity=20.32
- joint l_ankle_roll: limit lower=-0.44 upper=0.44 effort=3 velocity=20.32 -> lower=-0.44 upper=0.44 effort=8 velocity=20.32; type revolute -> fixed
- joint l_elbow_pitch: limit lower=-2.27 upper=2.27 effort=30 velocity=7.33 -> lower=-2.27 upper=2.27 effort=18 velocity=7.33; origin xyz=0 1.28869477361571E-05 -0.188546025627068 rpy=0 0 0 -> xyz=0 1.28869477361571E-05 -0.188546025627068 rpy=0 -0.3 0
- joint l_hip_pitch: limit lower=-1.75 upper=0.7 effort=160 velocity=37.38 -> lower=-1.75 upper=0.7 effort=130 velocity=37.38
- joint l_hip_roll: limit lower=-0.09 upper=0.79 effort=100 velocity=12.15 -> lower=-0.09 upper=0.79 effort=60 velocity=12.15
- joint l_hip_yaw: limit lower=-0.7 upper=0.7 effort=82.5 velocity=16.76 -> lower=-0.7 upper=0.7 effort=45 velocity=16.76
- joint l_knee_pitch: limit lower=-0.09 upper=1.92 effort=160 velocity=37.38 -> lower=-0.09 upper=1.92 effort=130 velocity=37.38
- joint l_shoulder_pitch: limit lower=-2.79 upper=1.92 effort=38 velocity=9.11 -> lower=-2.79 upper=1.92 effort=18 velocity=9.11; type revolute -> fixed
- joint l_shoulder_roll: limit lower=-0.57 upper=3.27 effort=38 velocity=9.11 -> lower=-0.57 upper=3.27 effort=18 velocity=9.11; origin xyz=0 0.067 0 rpy=-0.1364 0 0 -> xyz=0 0.067 0 rpy=-0.2364 0 0
- joint l_shoulder_yaw: limit lower=-2.97 upper=2.97 effort=30 velocity=7.33 -> lower=-2.97 upper=2.97 effort=18 velocity=7.33
- joint r_ankle_pitch: limit lower=-1.05 upper=0.52 effort=8 velocity=20.32 -> lower=-1.05 upper=0.52 effort=16 velocity=20.32
- joint r_ankle_roll: limit lower=-0.44 upper=0.44 effort=3 velocity=20.32 -> lower=-0.44 upper=0.44 effort=8 velocity=20.32; type revolute -> fixed
- joint r_elbow_pitch: limit lower=-2.27 upper=2.27 effort=30 velocity=7.33 -> lower=-2.27 upper=2.27 effort=18 velocity=7.33; origin xyz=0 1.28858724863512E-05 -0.188530329837713 rpy=0 0 0 -> xyz=0 1.28858724863512E-05 -0.188530329837713 rpy=0 -0.3 0
- joint r_hip_pitch: limit lower=-1.75 upper=0.7 effort=160 velocity=37.38 -> lower=-1.75 upper=0.7 effort=130 velocity=37.38
- joint r_hip_roll: limit lower=-0.79 upper=0.09 effort=100 velocity=12.15 -> lower=-0.79 upper=0.09 effort=60 velocity=12.15
- joint r_hip_yaw: limit lower=-0.7 upper=0.7 effort=82.5 velocity=16.76 -> lower=-0.7 upper=0.7 effort=45 velocity=16.76
- joint r_knee_pitch: limit lower=-0.09 upper=1.92 effort=160 velocity=37.38 -> lower=-0.09 upper=1.92 effort=130 velocity=37.38
- joint r_shoulder_pitch: limit lower=-2.79 upper=1.92 effort=38 velocity=9.11 -> lower=-2.79 upper=1.92 effort=18 velocity=9.11; type revolute -> fixed
- joint r_shoulder_roll: limit lower=-3.27 upper=0.57 effort=38 velocity=9.11 -> lower=-3.27 upper=0.57 effort=18 velocity=9.11; origin xyz=0 -0.067 0 rpy=0.13627 0 0 -> xyz=0 -0.067 0 rpy=0.23627 0 0
- joint r_shoulder_yaw: limit lower=-2.97 upper=2.97 effort=30 velocity=7.33 -> lower=-2.97 upper=2.97 effort=18 velocity=7.33
- joint waist_pitch: limit lower=-0.52 upper=1.22 effort=82.5 velocity=16.76 -> lower=-0.52 upper=1.22 effort=45 velocity=16.76; type revolute -> fixed
- joint waist_roll: limit lower=-0.7 upper=0.7 effort=82.5 velocity=16.76 -> lower=-0.7 upper=0.7 effort=45 velocity=16.76; type revolute -> fixed
- joint waist_yaw: limit lower=-1.05 upper=1.05 effort=82.5 velocity=16.76 -> lower=-1.05 upper=1.05 effort=45 velocity=16.76; type revolute -> fixed
