Commit message: refine code

File: legged_gym/resources/robots/GR1T1/urdf/GR1T1_lower_limb.urdf (robot description, URDF)
Before this commit: robot GR1T1, 34 links, 33 joints
Joints:
- joint l_hip_roll: limit lower=-0.09 upper=0.79 effort=60 velocity=12.15 -> lower=-0.09 upper=0.79 effort=40 velocity=12.15
- joint r_hip_roll: limit lower=-0.79 upper=0.09 effort=60 velocity=12.15 -> lower=-0.79 upper=0.09 effort=40 velocity=12.15

Commit message: refine code

File: legged_gym/resources/robots/GR1T1/urdf/GR1T1_lower_limb.urdf (robot description, URDF)
Before this commit: robot GR1T1, 34 links, 33 joints
Joints:
- joint head_pitch: axis 0 1 6.8349E-05 -> 0 1 0
- joint head_yaw: axis -1.221E-05 -6.8349E-05 1 -> 0 0 1
- joint l_ankle_pitch: limit lower=-1.05 upper=0.52 effort=16 velocity=20.32 -> lower=-1.05 upper=0.52 effort=18 velocity=20.32
- joint l_ankle_roll: axis 1 0 1.221E-05 -> 1 0 0; limit lower=-0.44 upper=0.44 effort=8 velocity=20.32 -> lower=-0.44 upper=0.44 effort=9 velocity=20.32
- joint l_elbow_pitch: axis 0 0.999999997664201 6.83490816804566E-05 -> 0 1 0; limit lower=-2.27 upper=2.27 effort=18 velocity=7.33 -> lower=-2.27 upper=2.27 effort=30 velocity=7.33
- joint l_hip_pitch: axis 0 1 -6.8349E-05 -> 0 1 0
- joint l_hip_roll: axis 1 0 1.221E-05 -> 1 0 0; origin xyz=-0.047999 0.105 -0.057493 rpy=0 0 0 -> xyz=-0.048 0.105 -0.0575 rpy=0 0 0
- joint l_shoulder_pitch: limit lower=-2.79 upper=1.92 effort=18 velocity=9.11 -> lower=-2.79 upper=1.92 effort=30 velocity=9.11
- joint l_shoulder_roll: axis 1 0 -1.221E-05 -> 1 0 0; limit lower=-0.57 upper=3.27 effort=18 velocity=9.11 -> lower=-0.57 upper=3.27 effort=30 velocity=9.11
- joint l_shoulder_yaw: axis 1.221E-05 6.8349E-05 1 -> 0 0 1; limit lower=-2.97 upper=2.97 effort=18 velocity=7.33 -> lower=-2.97 upper=2.97 effort=30 velocity=7.33
- joint l_wrist_pitch: axis 0 1 6.8349E-05 -> 0 1 0
- joint l_wrist_yaw: axis 1.22100045815953E-05 6.83490816738029E-05 0.999999997589659 -> 0 0 1
- joint r_ankle_pitch: axis 0 1 6.8349E-05 -> 0 1 0; limit lower=-1.05 upper=0.52 effort=16 velocity=20.32 -> lower=-1.05 upper=0.52 effort=18 velocity=20.32; origin xyz=0 2.3239E-05 -0.34 rpy=0 0 0 -> xyz=0 0 -0.34 rpy=0 0 0
- joint r_ankle_roll: axis 1 0 1.221E-05 -> 1 0 0; limit lower=-0.44 upper=0.44 effort=8 velocity=20.32 -> lower=-0.44 upper=0.44 effort=9 velocity=20.32
- joint r_elbow_pitch: axis 0 0.999999997664136 -6.83500416450034E-05 -> 0 1 0; limit lower=-2.27 upper=2.27 effort=18 velocity=7.33 -> lower=-2.27 upper=2.27 effort=30 velocity=7.33
- joint r_hip_pitch: axis 0 1 6.8349E-05 -> 0 1 0
- joint r_hip_roll: axis 1 0 1.221E-05 -> 1 0 0; origin xyz=-0.047999 -0.105 -0.057508 rpy=0 0 0 -> xyz=-0.048 -0.105 -0.0575 rpy=0 0 0
- joint r_hip_yaw: axis 1.2209E-05 6.8349E-05 1 -> 0 0 1; origin xyz=0.048 0 -0.030499 rpy=0 0 0 -> xyz=0.048 0 -0.0305 rpy=0 0 0
- joint r_knee_pitch: axis 0 1 -6.8349E-05 -> 0 1 0; origin xyz=0 2.4606E-05 -0.36 rpy=0 0 0 -> xyz=0 0 -0.36 rpy=0 0 0
- joint r_shoulder_pitch: limit lower=-2.79 upper=1.92 effort=18 velocity=9.11 -> lower=-2.79 upper=1.92 effort=30 velocity=9.11
- joint r_shoulder_roll: axis 1 0 -1.221E-05 -> 1 0 0; limit lower=-3.27 upper=0.57 effort=18 velocity=9.11 -> lower=-3.27 upper=0.57 effort=30 velocity=9.11
- joint r_shoulder_yaw: limit lower=-2.97 upper=2.97 effort=18 velocity=7.33 -> lower=-2.97 upper=2.97 effort=30 velocity=7.33
- joint r_wrist_pitch: axis 0 1 -6.835E-05 -> 0 1 0
- joint r_wrist_roll: axis 1 0 1.221E-05 -> 1 0 0
- joint waist_pitch: axis 0 1 -6.8349E-05 -> 0 1 0
- joint waist_roll: axis 1 0 1.221E-05 -> 1 0 0
- joint waist_yaw: axis -1.221E-05 -6.8349E-05 1 -> 0 0 1

File: legged_gym/resources/robots/GR1T2/urdf/GR1T2_lower_limb.urdf (robot description, URDF)
Before this commit: robot GR1T2, 35 links, 34 joints
Joints:
- joint joint_head_pitch: origin xyz=0.000999999999997045 -0.000225512658326668 0.144786985472057 rpy=0 0 0 -> xyz=0.000999999999997045 -0.000130512658326668 0.144786985472057 rpy=0 0 0
- joint l_ankle_pitch: limit lower=-1.05 upper=0.52 effort=15 velocity=20.32 -> lower=-1.05 upper=0.52 effort=18 velocity=20.32
- joint l_ankle_roll: limit lower=-0.44 upper=0.44 effort=30 velocity=20.32 -> lower=-0.44 upper=0.44 effort=9 velocity=20.32
- joint l_hip_pitch: limit lower=-1.75 upper=0.7 effort=225 velocity=37.38 -> lower=-1.75 upper=0.7 effort=130 velocity=37.38
- joint l_hip_roll: limit lower=-0.09 upper=0.79 effort=48 velocity=12.15 -> lower=-0.09 upper=0.79 effort=40 velocity=12.15; origin xyz=-0.0480000000000005 0.105 -0.0575 rpy=0 0 0 -> xyz=-0.048 0.105 -0.0575 rpy=0 0 0
- joint l_hip_yaw: limit lower=-0.7 upper=0.7 effort=66 velocity=16.76 -> lower=-0.7 upper=0.7 effort=45 velocity=16.76
- joint l_knee_pitch: limit lower=-0.09 upper=1.92 effort=225 velocity=37.38 -> lower=-0.09 upper=1.92 effort=130 velocity=37.38
- joint l_shoulder_pitch: limit lower=-2.79 upper=1.92 effort=38 velocity=9.11 -> lower=-2.79 upper=1.92 effort=30 velocity=9.11
- joint l_shoulder_roll: limit lower=-0.57 upper=3.27 effort=38 velocity=9.11 -> lower=-0.57 upper=3.27 effort=30 velocity=9.11
- joint r_ankle_pitch: limit lower=-1.05 upper=0.52 effort=15 velocity=20.32 -> lower=-1.05 upper=0.52 effort=18 velocity=20.32; origin xyz=0 0 -0.339999999788054 rpy=0 0 0 -> xyz=0 0 -0.34 rpy=0 0 0
- joint r_ankle_roll: limit lower=-0.44 upper=0.44 effort=30 velocity=20.32 -> lower=-0.44 upper=0.44 effort=9 velocity=20.32
- joint r_hip_pitch: limit lower=-1.75 upper=0.7 effort=225 velocity=37.38 -> lower=-1.75 upper=0.7 effort=130 velocity=37.38; origin xyz=0 0 -0.109999999999337 rpy=0 0 0 -> xyz=0 0 -0.11 rpy=0 0 0
- joint r_hip_roll: limit lower=-0.79 upper=0.09 effort=48 velocity=12.15 -> lower=-0.79 upper=0.09 effort=40 velocity=12.15; origin xyz=-0.0480000000000003 -0.105 -0.0575 rpy=0 0 0 -> xyz=-0.048 -0.105 -0.0575 rpy=0 0 0
- joint r_hip_yaw: limit lower=-0.7 upper=0.7 effort=66 velocity=16.76 -> lower=-0.7 upper=0.7 effort=45 velocity=16.76; origin xyz=0.0480000000000212 0 -0.0305000000000011 rpy=0 0 0 -> xyz=0.048 0 -0.0305 rpy=0 0 0
- joint r_knee_pitch: limit lower=-0.09 upper=1.92 effort=225 velocity=37.38 -> lower=-0.09 upper=1.92 effort=130 velocity=37.38; origin xyz=0 0 -0.359995124115985 rpy=0 0 0 -> xyz=0 0 -0.36 rpy=0 0 0
- joint r_shoulder_pitch: limit lower=-2.79 upper=1.92 effort=38 velocity=9.11 -> lower=-2.79 upper=1.92 effort=30 velocity=9.11
- joint r_shoulder_roll: limit lower=-3.27 upper=0.57 effort=38 velocity=9.11 -> lower=-3.27 upper=0.57 effort=30 velocity=9.11
- joint waist_pitch: limit lower=-0.52 upper=1.22 effort=66 velocity=16.76 -> lower=-0.52 upper=1.22 effort=45 velocity=16.76; origin xyz=0 0 0.0570000000000001 rpy=0 0 0 -> xyz=0 0 0.057 rpy=0 0 0
- joint waist_roll: limit lower=-0.7 upper=0.7 effort=66 velocity=16.76 -> lower=-0.7 upper=0.7 effort=45 velocity=16.76
- joint waist_yaw: limit lower=-1.05 upper=1.05 effort=66 velocity=16.76 -> lower=-1.05 upper=1.05 effort=45 velocity=16.76; origin xyz=0 0 0.00649999999999984 rpy=0 0 0 -> xyz=0 0 0.0065 rpy=0 0 0

Commit message: refine GR1T1_lower_limb.urdf and GR1T2_lower_limb.urdf to make bend elbow posture

File: legged_gym/resources/robots/GR1T1/urdf/GR1T1_lower_limb.urdf (robot description, URDF)
Before this commit: robot GR1T1, 37 links, 36 joints
Joints:
- joint left_elbow_pitch_joint: origin xyz=0 0 -0.1751 rpy=0 0 0 -> xyz=0 0 -0.1751 rpy=0 -0.3 0
- joint left_shoulder_roll_joint: origin xyz=0 0.09515 0 rpy=-0.43633 0 0 -> xyz=0 0.09515 0 rpy=-0.23633 0 0
- joint right_elbow_pitch_joint: origin xyz=0 0 -0.1751 rpy=0 0 0 -> xyz=0 0 -0.1751 rpy=0 -0.3 0
- joint right_shoulder_roll_joint: origin xyz=0 -0.09515 0 rpy=0.43633 0 0 -> xyz=0 -0.09515 0 rpy=0.23633 0 0

File: legged_gym/resources/robots/GR1T2/urdf/GR1T2_lower_limb.urdf (robot description, URDF)
Before this commit: robot GR1T2, 37 links, 36 joints
Joints:
- joint left_elbow_pitch_joint: origin xyz=0 0.0010503 -0.1786 rpy=0 0 0 -> xyz=0 0.0010503 -0.1786 rpy=0 -0.3 0
- joint left_shoulder_roll_joint: origin xyz=0 0.09515 0 rpy=-0.43275 0 0 -> xyz=0 0.09515 0 rpy=-0.23275 0 0
- joint right_elbow_pitch_joint: origin xyz=0 -0.0010503 -0.1786 rpy=0 0 0 -> xyz=0 -0.0010503 -0.1786 rpy=0 -0.3 0
- joint right_shoulder_roll_joint: origin xyz=0 -0.09515 0 rpy=0.43275 0 0 -> xyz=0 -0.09515 0 rpy=0.23275 0 0
