Commit message: refine code and URDF files

File: legged_gym/resources/robots/GR1T1/urdf/GR1T1.urdf (robot description, URDF)
Before this commit: robot GR1T1, 37 links, 36 joints
Joints:
- joint left_hip_pitch_joint: limit lower=-1.75 upper=0.7 effort=225 velocity=37.38 -> lower=-1.75 upper=0.7 effort=130 velocity=37.38
- joint left_knee_pitch_joint: limit lower=-0.09 upper=1.92 effort=225 velocity=37.38 -> lower=-0.09 upper=1.92 effort=130 velocity=37.38
- joint right_hip_pitch_joint: limit lower=-1.75 upper=0.7 effort=225 velocity=37.38 -> lower=-1.75 upper=0.7 effort=130 velocity=37.38
- joint right_knee_pitch_joint: limit lower=-0.09 upper=1.92 effort=225 velocity=37.38 -> lower=-0.09 upper=1.92 effort=130 velocity=37.38

File: legged_gym/resources/robots/GR1T1/urdf/GR1T1_lower_limb.urdf (robot description, URDF)
Before this commit: robot GR1T1, 37 links, 36 joints
Joints:
- joint left_hip_pitch_joint: limit lower=-1.75 upper=0.7 effort=225 velocity=37.38 -> lower=-1.75 upper=0.7 effort=130 velocity=37.38
- joint left_knee_pitch_joint: limit lower=-0.09 upper=1.92 effort=225 velocity=37.38 -> lower=-0.09 upper=1.92 effort=130 velocity=37.38
- joint right_hip_pitch_joint: limit lower=-1.75 upper=0.7 effort=225 velocity=37.38 -> lower=-1.75 upper=0.7 effort=130 velocity=37.38
- joint right_knee_pitch_joint: limit lower=-0.09 upper=1.92 effort=225 velocity=37.38 -> lower=-0.09 upper=1.92 effort=130 velocity=37.38

File: legged_gym/resources/robots/GR1T2/urdf/GR1T2.urdf (robot description, URDF)
Before this commit: robot GR1T2, 37 links, 36 joints
Joints:
- joint left_hip_pitch_joint: limit lower=-1.75 upper=0.7 effort=225 velocity=37.38 -> lower=-1.75 upper=0.7 effort=130 velocity=37.38
- joint left_knee_pitch_joint: limit lower=-0.09 upper=1.92 effort=225 velocity=37.38 -> lower=-0.09 upper=1.92 effort=130 velocity=37.38
- joint right_hip_pitch_joint: limit lower=-1.75 upper=0.7 effort=225 velocity=37.38 -> lower=-1.75 upper=0.7 effort=130 velocity=37.38
- joint right_knee_pitch_joint: limit lower=-0.09 upper=1.92 effort=225 velocity=37.38 -> lower=-0.09 upper=1.92 effort=130 velocity=37.38

File: legged_gym/resources/robots/GR1T2/urdf/GR1T2_lower_limb.urdf (robot description, URDF)
Before this commit: robot GR1T2, 37 links, 36 joints
Joints:
- joint left_hip_pitch_joint: limit lower=-1.75 upper=0.7 effort=225 velocity=37.38 -> lower=-1.75 upper=0.7 effort=130 velocity=37.38
- joint left_knee_pitch_joint: limit lower=-0.09 upper=1.92 effort=225 velocity=37.38 -> lower=-0.09 upper=1.92 effort=130 velocity=37.38
- joint right_hip_pitch_joint: limit lower=-1.75 upper=0.7 effort=225 velocity=37.38 -> lower=-1.75 upper=0.7 effort=130 velocity=37.38
- joint right_knee_pitch_joint: limit lower=-0.09 upper=1.92 effort=225 velocity=37.38 -> lower=-0.09 upper=1.92 effort=130 velocity=37.38
